File: AgnusAdaptor.sch (EAGLE design)
At the start: 5 parts, among them IC1 AGNUS_8375_A500+_A600_THT, IC3 74LS02D

Commit message: first go at routing complete
Parts:
- added JP1: RAS jumpers, pinhead:PINHD-1X3
- C2: value (none) -> 100uF
- IC2: value (none) -> A3000 Agnus Socket
Connections:
- net !RAS: now also JP1.3
- net !RAS0: now also IC3A.I1, JP1.1; no longer IC3A.I0
- net !RAS1: now also IC3A.I0, JP1.2; no longer IC3A.I1
- net GND: now also IC3C.I0, IC3C.I1, IC3D.I0, IC3D.I1
Other:
- moved on the sheet: IC3A, IC3B
