File: AgnusAdaptor.brd (EAGLE design)
At the start: 53.3 x 78.7 mm, 5 parts, among them IC1 AGNUS_8375_A500+_A600_THT, IC3 74LS02D

Commit message: first go at routing complete
Parts:
- added JP1: RAS jumpers, pinhead:1X03
- C2: value (none) -> 100uF
- IC2: value (none) -> A3000 Agnus Socket
- moved C1 5.34 mm to (46.0, 40.4)
- turned C2 to 0 degrees
Connections:
- new net S$1: IC2.25
- net !RAMEN: no longer IC2.25
- net !RAS: now also JP1.3
- net !RAS0: now also IC3.3, JP1.1; no longer IC3.2
- net !RAS1: now also IC3.2, JP1.2; no longer IC3.3
- net GND: now also IC3.11, IC3.12, IC3.8, IC3.9
Routing:
- net RGA2: track 0.00 -> 133.3 mm, vias 0 -> 1
- net RGA4: track 0.00 -> 126.0 mm, vias 0 -> 1
- net RGA3: track 0.00 -> 124.1 mm
- net RGA5: track 0.00 -> 122.9 mm
- net RGA6: track 0.00 -> 121.5 mm
- net !AS: track 0.00 -> 105.9 mm
- net !RAMEN: track 0.00 -> 101.5 mm
- net !WE: track 0.00 -> 89.0 mm
- net !BLISS: track 0.00 -> 82.6 mm
- net RGA8: track 0.00 -> 71.7 mm
- net DRA9: track 0.00 -> 58.9 mm
- net DRA7: track 0.00 -> 58.6 mm
- net VCC: track 96.3 -> 154.5 mm, vias 0 -> 2
- net DRA5: track 0.00 -> 57.0 mm
- net DRD7: track 0.00 -> 56.2 mm
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Other:
- board text added: "A3000 Agnus Adapter Prototype V0.1"
- board text removed: "A3000 Agnus Adapter"

Commit message: fixed back annotation issue in board and added docs and libs
Connections:
- removed net S$1: IC2.25
- net !RAMEN: now also IC2.25
Routing:
- net !RAMEN: track 101.5 -> 110.3 mm
- net S$1: track 1.86 -> 0.00 mm
Changed lines of the file:
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@@
 <wire x1="50.038" y1="64.50868125" x2="50.038" y2="28.702" width="0.1524" layer="16"/>
-</signal>
-<signal name="S$1">
-<contactref element="IC2" pad="25"/>
-<wire x1="22.352" y1="75.692" x2="22.8473" y2="76.1873" width="0.15" layer="16"/>
-<wire x1="22.8473" y1="76.1873" x2="24.003" y2="76.1873" width="0.15" layer="16"/>
 </signal>
 <signal name="!RAMEN">
 <contactref element="IC1" pad="25"/>
+<contactref element="IC2" pad="25"/>
 <wire x1="28.8925" y1="95.7453" x2="28.1813" y2="96.4565" width="0.15" layer="16"/>
-<wire x1="28.8925" y1="81.0768" x2="28.8925" y2="95.7453" width="0.15" layer="16"/>
+<wire x1="28.8925" y1="81.1657" x2="28.8925" y2="95.7453" width="0.15" layer="16"/>
 <wire x1="28.1813" y1="96.4565" x2="10.668" y2="96.4565" width="0.15" layer="16"/>
 <wire x1="3.2893" y1="37.6936" x2="5.1562" y2="35.8267" width="0.15" layer="16"/>
@@
 <wire x1="3.2893" y1="89.0778" x2="3.2893" y2="37.6936" width="0.15" layer="16"/>
 <wire x1="7.3787" y1="35.8267" x2="8.382" y2="36.83" width="0.15" layer="16"/>
+<wire x1="28.8925" y1="81.1657" x2="28.0924" y2="80.3656" width="0.1524" layer="16"/>
+<wire x1="28.0924" y1="80.3656" x2="23.4188" y2="75.692" width="0.1524" layer="16"/>
+<wire x1="22.352" y1="75.692" x2="23.4188" y2="75.692" width="0.1524" layer="16"/>
 </signal>
 <signal name="!REGEN">
